File: hw/softtag.sch (KiCad schematic (older format))
At the start: 20 parts, among them P1 CONN_01X06, Q1 Q_NMOS_GSD, U1 PIC12LF1612-E/SN

Commit message: Update the schematic
Parts:
- removed C2: CTRIM, Capacitors_SMD:C_1206_HandSoldering, symbol CTRIM
- removed R6: R, Resistors_SMD:R_0805, symbol R
- added C2, C6: C, Capacitors_SMD:C_0805, symbol C
- added D5: 1N4148, symbol D
- C3: value C -> 22pF
- C4: value CP -> 22nF
- D1: value D_Schottky -> BAT85
- D2: value D -> 1N4148
- D3, D4: value ZENER -> 3V3
- R8: renamed from R?; value R -> 330k
Connections:
- wire segments 77 -> 99
Other:
- note added: "PCB Inductor\n1 µH"
- note removed: "PCB Inductor"
- moved on the sheet: C1, C5, D1, D4, R7

Commit message: update schematic
Parts:
- C1: value C -> 100pF
- C2: value C -> 33pF
- C4: value 22nF -> 22uF
- C6: value C -> 10pF
- R1, R3: value R -> 1M
- R2: value R -> 100k
Changed lines of the file:
@@
 P 2300 2250
 F 0 "C1" H 2200 2350 50  0000 L CNN
-F 1 "C" H 2350 2350 50  0000 L CNN
+F 1 "100pF" H 2350 2350 50  0000 L CNN
 F 2 "Capacitors_SMD:C_0805" H 2338 2100 50  0001 C CNN
 F 3 "" H 2300 2250 50  0000 C CNN
@@
 P 4750 1150
 F 0 "R2" H 4820 1196 50  0000 L CNN
-F 1 "R" H 4820 1105 50  0000 L CNN
+F 1 "100k" H 4820 1105 50  0000 L CNN
 F 2 "Resistors_SMD:R_0805" V 4680 1150 50  0001 C CNN
 F 3 "" H 4750 1150 50  0000 C CNN
@@
 P 4750 2250
 F 0 "R3" H 4820 2296 50  0000 L CNN
-F 1 "R" H 4820 2205 50  0000 L CNN
+F 1 "1M" H 4820 2205 50  0000 L CNN
 F 2 "Resistors_SMD:R_0805" V 4680 2250 50  0001 C CNN
 F 3 "" H 4750 2250 50  0000 C CNN
@@
 P 3650 2400
 F 0 "R1" H 3700 2450 50  0000 L CNN
-F 1 "R" H 3720 2355 50  0000 L CNN
+F 1 "1M" H 3720 2355 50  0000 L CNN
 F 2 "Resistors_SMD:R_0805" V 3580 2400 50  0001 C CNN
 F 3 "" H 3650 2400 50  0000 C CNN
@@
 P 4450 2250
 F 0 "C4" H 4568 2296 50  0000 L CNN
-F 1 "22nF" H 4568 2205 30  0000 L CNN
+F 1 "22uF" H 4568 2205 30  0000 L CNN
 F 2 "Capacitors_Tantalum_SMD:TantalC_SizeA_EIA-3216_HandSoldering" H 4488 2100 50  0001 C CNN
 F 3 "" H 4450 2250 50  0000 C CNN
@@
 P 2600 2250
 F 0 "C2" H 2500 2350 50  0000 L CNN
-F 1 "C" H 2650 2350 50  0000 L CNN
+F 1 "33pF" H 2650 2350 50  0000 L CNN
 F 2 "Capacitors_SMD:C_0805" H 2638 2100 50  0001 C CNN
 F 3 "" H 2600 2250 50  0000 C CNN
@@
 P 2900 2250
 F 0 "C6" H 2800 2350 50  0000 L CNN
-F 1 "C" H 2950 2350 50  0000 L CNN
+F 1 "10pF" H 2950 2350 50  0000 L CNN
 F 2 "Capacitors_SMD:C_0805" H 2938 2100 50  0001 C CNN
 F 3 "" H 2900 2250 50  0000 C CNN
