File: hw/softtag.sch (KiCad schematic (older format))
At the start: 21 parts, among them P1 CONN_01X06, Q1 Q_NMOS_GSD, U1 PIC12LF1612-E/SN

Commit message: updated schematic
Parts:
- removed P1: CONN_01X06, Pin_Headers:Pin_Header_Straight_1x06, symbol CONN_01X06
- added C10, C8, C9: 100n, symbol C
- added C7: 1n, Capacitors_SMD:C_0805, symbol C
- added R6: 1k, symbol R
- added U2: MMA7260QT, symbol MMA7260QT
- C5: value C -> 100n
- R4, R5: value R -> 1k; footprint Resistors_SMD:R_0805 -> (none)
Connections:
- net labels added: ACC_X, ACC_Y, ACC_Z
- net labels removed: FREE0, FREE1, FREE2, FREE3
- wire segments 99 -> 79
- no-connect marks 0 -> 1
Other:
- moved on the sheet: C5, U1
